Commit message: Update robot to 4 DoF and add automated Python trajectory publisher

File: src/my_first/urdf/my_robot.urdf (robot description, URDF)
Before this commit: robot test_robot, 1 links, 0 joints
Links:
- added link arm_1_link; collision cylinder length=0.5 radius=0.05; visual cylinder length=0.5 radius=0.05
- added link arm_2_link; collision cylinder length=0.5 radius=0.05; visual cylinder length=0.5 radius=0.05
- added link arm_3_link; collision cylinder length=0.5 radius=0.05; visual cylinder length=0.5 radius=0.05
- added link gripper_left_link; collision box size=0.04 0.02 0.08; visual box size=0.04 0.02 0.08
- added link gripper_right_link; collision box size=0.04 0.02 0.08; visual box size=0.04 0.02 0.08
- added link hand_link; collision box size=0.06 0.2 0.05; visual box size=0.06 0.2 0.05
- link base_link: geometry collision box size=0.2 0.2 0.3; visual box size=0.2 0.2 0.3
Joints:
- added joint arm_0_joint: type revolute, parent base_link, child arm_1_link, origin xyz=0 0 0.15 rpy=0 0 0, axis 0 0 1, limit lower=-3.14 upper=3.14 effort=10.0 velocity=1.0
- added joint arm_1_joint: type revolute, parent arm_1_link, child arm_2_link, origin xyz=0 0 0.5 rpy=0 0 0, axis 0 1 0, limit lower=-1.57 upper=1.57 effort=10.0 velocity=1.0
- added joint arm_2_joint: type revolute, parent arm_2_link, child arm_3_link, origin xyz=0 0 0.5 rpy=0 0 0, axis 0 1 0, limit lower=-1.57 upper=1.57 effort=10.0 velocity=1.0
- added joint arm_3_joint: type revolute, parent arm_3_link, child hand_link, origin xyz=0 0 0.5 rpy=0 0 0, axis 0 1 0, limit lower=-1.57 upper=1.57 effort=10.0 velocity=1.0
- added joint gripper_1_joint: type prismatic, parent hand_link, child gripper_left_link, origin xyz=0 0.08 0.05 rpy=0 0 0, axis 0 -1 0, limit lower=0.0 upper=0.06 effort=5.0 velocity=0.5
- added joint gripper_2_joint: type prismatic, parent hand_link, child gripper_right_link, origin xyz=0 -0.08 0.05 rpy=0 0 0, axis 0 1 0, limit lower=0.0 upper=0.06 effort=5.0 velocity=0.5

Commit message: fix: resolve joint_state_broadcaster issue and add ch7 moveit gazebo launch

File: src/my_first/urdf/my_robot.urdf (robot description, URDF)
Before this commit: robot test_robot, 7 links, 6 joints
Links:
- link arm_1_link: mass None -> 1.0
- link arm_2_link: mass None -> 1.0
- link arm_3_link: mass None -> 1.0
- link base_link: mass None -> 50.0
- link gripper_left_link: mass None -> 0.2
- link gripper_right_link: mass None -> 0.2
- link hand_link: mass None -> 0.5
